File: i2c.brd (EAGLE design)
At the start: 36.5 x 34.3 mm, 7 parts, among them IC1 24LC024SN, IC2 24LC024ST, X1 2510-

Commit message: Добавлена надпись
Routing:
- net GND: track 124.6 -> 94.1 mm
Other:
- board text added: "I2C 24"
Changed lines of the file:
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@@
 <layer number="40" name="bKeepout" color="1" fill="11" visible="no" active="yes"/>
 <layer number="41" name="tRestrict" color="4" fill="10" visible="no" active="yes"/>
-<layer number="42" name="bRestrict" color="1" fill="10" visible="no" active="yes"/>
+<layer number="42" name="bRestrict" color="1" fill="10" visible="yes" active="yes"/>
 <layer number="43" name="vRestrict" color="2" fill="10" visible="no" active="yes"/>
 <layer number="44" name="Drills" color="7" fill="1" visible="no" active="yes"/>
@@
 <vertex x="58.42" y="44.45"/>
 </polygon>
+<polygon width="0.2" layer="42">
+<vertex x="45.72" y="63.5"/>
+<vertex x="57.15" y="63.5"/>
+<vertex x="57.15" y="58.42"/>
+<vertex x="45.72" y="58.42"/>
+</polygon>
+<text x="54.61" y="59.69" size="1.778" layer="16" rot="MR0">I2C 24</text>
 </plain>
 <attributes>
@@
 <wire x1="40.64" y1="41.25" x2="40.64" y2="43.18" width="0.254" layer="16"/>
 <wire x1="50.86" y1="44.45" x2="52.07" y2="44.45" width="0.254" layer="16"/>
-<wire x1="55.88" y1="44.45" x2="55.88" y2="60.96" width="0.254" layer="16"/>
-<wire x1="55.88" y1="60.96" x2="41.91" y2="60.96" width="0.254" layer="16"/>
 <wire x1="39.37" y1="60.96" x2="41.91" y2="60.96" width="0.508" layer="16"/>
 <wire x1="36.83" y1="60.96" x2="39.37" y2="60.96" width="0.508" layer="16"/>
@@
 <wire x1="52.07" y1="44.45" x2="54.61" y2="44.45" width="0.508" layer="16"/>
 <wire x1="54.61" y1="44.45" x2="55.88" y2="44.45" width="0.508" layer="16"/>
+<wire x1="38.0765" y1="47.0135" x2="36.83" y2="60.96" width="0" layer="19" extent="16-16"/>
 </signal>
 <signal name="RST">
